File: chastityRightV2/chastityRightV2.kicad_sch (KiCad schematic)
At the start: 260 parts, among them J1 Conn_01x04, J2 USB_C_Receptacle_USB2.0, J3 AudioJack3, J4 Conn_01x05, J6 USB_C_Receptacle_USB2.0, J7 Conn_01x04, J8 Conn_01x05, SW2 RotaryEncoder_Switch, U1 XC6206PxxxMR, U2 SRV05-4, U3 RP2040, U4 W25Q128JVS, U5 XC6206PxxxMR, U6 SRV05-4, U7 W25Q128JVS, U8 RP2040, Y1 Crystal_GND24, Y2 Crystal_GND24

Commit message: Add files via upload
Parts:
- added C33: 100n, Capacitor_SMD:C_0402_1005Metric, symbol Device:C_Small
- added C34, C35, C36, C37, C38: 100u, Capacitor_SMD:C_0402_1005Metric, symbol Device:C_Small
- added C39: 100n, Capacitor_SMD:C_0805_2012Metric, symbol Device:C
- added R19, R20: 5.1k, Resistor_SMD:R_0805_2012Metric, symbol Device:R
- added R21: 75k, Resistor_SMD:R_0805_2012Metric, symbol Device:R
- added U10: TPS2553DBVR, Package_TO_SOT_SMD:SOT-23-6, symbol Ghoul:TPS2553DBVR
- added U9: 74AHC1G125, SN74AHC1G125DRLR:DRL5, symbol 74xGxx:74AHC1G125
- LED1: renamed from D64; value WS2812B -> SK6803MINI-E
- LED10: renamed from D73; value WS2812B -> SK6803MINI-E
- LED11: renamed from D74; value WS2812B -> SK6803MINI-E
- LED12: renamed from D75; value WS2812B -> SK6803MINI-E
- LED13: renamed from D76; value WS2812B -> SK6803MINI-E
- LED14: renamed from D77; value WS2812B -> SK6803MINI-E
- LED15: renamed from D78; value WS2812B -> SK6803MINI-E
- LED16: renamed from D79; value WS2812B -> SK6803MINI-E
- LED17: renamed from D80; value WS2812B -> SK6803MINI-E
- LED18: renamed from D81; value WS2812B -> SK6803MINI-E
- LED19: renamed from D82; value WS2812B -> SK6803MINI-E
- LED2: renamed from D65; value WS2812B -> SK6803MINI-E
- LED20: renamed from D83; value WS2812B -> SK6803MINI-E
- LED21: renamed from D84; value WS2812B -> SK6803MINI-E
- LED22: renamed from D85; value WS2812B -> SK6803MINI-E
- LED23: renamed from D86; value WS2812B -> SK6803MINI-E
- LED24: renamed from D87; value WS2812B -> SK6803MINI-E
- LED25: renamed from D88; value WS2812B -> SK6803MINI-E
- LED26: renamed from D89; value WS2812B -> SK6803MINI-E
- LED27: renamed from D90; value WS2812B -> SK6803MINI-E
- LED28: renamed from D91; value WS2812B -> SK6803MINI-E
- LED29: renamed from D92; value WS2812B -> SK6803MINI-E
- LED3: renamed from D66; value WS2812B -> SK6803MINI-E
- LED30: renamed from D93; value WS2812B -> SK6803MINI-E
- LED31: renamed from D94; value WS2812B -> SK6803MINI-E
- LED32: renamed from D95; value WS2812B -> SK6803MINI-E
- LED33: renamed from D96; value WS2812B -> SK6803MINI-E
- LED34: renamed from D97; value WS2812B -> SK6803MINI-E
- LED35: renamed from D98; value WS2812B -> SK6803MINI-E
- LED36: renamed from D99; value WS2812B -> SK6803MINI-E
- LED37: renamed from D100; value WS2812B -> SK6803MINI-E
- LED38: renamed from D101; value WS2812B -> SK6803MINI-E
- LED39: renamed from D102; value WS2812B -> SK6803MINI-E
- LED4: renamed from D67; value WS2812B -> SK6803MINI-E
- LED40: renamed from D103; value WS2812B -> SK6803MINI-E
- LED41: renamed from D104; value WS2812B -> SK6803MINI-E
- LED42: renamed from D105; value WS2812B -> SK6803MINI-E
- LED43: renamed from D106; value WS2812B -> SK6803MINI-E
- LED44: renamed from D107; value WS2812B -> SK6803MINI-E
- LED45: renamed from D108; value WS2812B -> SK6803MINI-E
- LED46: renamed from D109; value WS2812B -> SK6803MINI-E
- LED47: renamed from D110; value WS2812B -> SK6803MINI-E
- LED48: renamed from D111; value WS2812B -> SK6803MINI-E
- LED49: renamed from D112; value WS2812B -> SK6803MINI-E
- LED5: renamed from D68; value WS2812B -> SK6803MINI-E
- LED50: renamed from D113; value WS2812B -> SK6803MINI-E
- LED51: renamed from D114; value WS2812B -> SK6803MINI-E
- LED52: renamed from D115; value WS2812B -> SK6803MINI-E
- LED53: renamed from D116; value WS2812B -> SK6803MINI-E
- LED54: renamed from D117; value WS2812B -> SK6803MINI-E
- LED55: renamed from D118; value WS2812B -> SK6803MINI-E
- LED56: renamed from D119; value WS2812B -> SK6803MINI-E
- LED57: renamed from D120; value WS2812B -> SK6803MINI-E
- LED58: renamed from D121; value WS2812B -> SK6803MINI-E
- LED59: renamed from D122; value WS2812B -> SK6803MINI-E
- LED6: renamed from D69; value WS2812B -> SK6803MINI-E
- LED60: renamed from D123; value WS2812B -> SK6803MINI-E
- LED7: renamed from D70; value WS2812B -> SK6803MINI-E
- LED8: renamed from D71; value WS2812B -> SK6803MINI-E
- LED9: renamed from D72; value WS2812B -> SK6803MINI-E
Connections:
- net +3V3: now also LED1.1 (VDD), LED10.1 (VDD), LED11.1 (VDD), LED12.1 (VDD), LED13.1 (VDD), LED14.1 (VDD), LED15.1 (VDD), LED16.1 (VDD), LED17.1 (VDD), LED18.1 (VDD), LED19.1 (VDD), LED2.1 (VDD), LED20.1 (VDD), LED21.1 (VDD), LED22.1 (VDD), LED23.1 (VDD), LED24.1 (VDD), LED25.1 (VDD), LED26.1 (VDD), LED27.1 (VDD), LED28.1 (VDD), LED29.1 (VDD), LED3.1 (VDD), LED30.1 (VDD), LED4.1 (VDD), LED5.1 (VDD), LED6.1 (VDD), LED7.1 (VDD), LED8.1 (VDD), LED9.1 (VDD)
- net +5V: now also C33.2, C39.1, R19.1, U10.1 (IN), U9.5 (VCC)
- net GND: now also C33.1, C34.1, C35.1, C36.1, C37.1, C38.1, C39.2, R20.2, R21.2, U10.2 (GND), U9.1, U9.3 (GND)
- net LED_Data: no longer LED55.3 (DIN)
- net at LED42.3 (DIN): now also LED36.2 (DOUT); no longer LED48.2 (DOUT)
- net at LED60.2 (DOUT): no longer LED54.3 (DIN)
- net at LED37.2 (DOUT): now also LED43.3 (DIN); no longer LED31.3 (DIN)
- net LED_Data_3V3: now reaches U3.39 (GPIO27_ADC1)
- net LED_Data_3V3: now also U9.2
- net at LED49.2 (DOUT): now also LED55.3 (DIN); no longer LED43.3 (DIN)
- net VCC renamed LED_Pow_5V
- net LED_Pow_5V: now also C34.2, C35.2, C36.2, C37.2, C38.2, U10.6 (OUT); no longer LED1.1 (VDD), LED10.1 (VDD), LED11.1 (VDD), LED12.1 (VDD), LED19.1 (VDD), LED2.1 (VDD), LED20.1 (VDD), LED21.1 (VDD), LED22.1 (VDD), LED23.1 (VDD), LED24.1 (VDD), LED25.1 (VDD), LED26.1 (VDD), LED27.1 (VDD), LED28.1 (VDD), LED29.1 (VDD), LED3.1 (VDD), LED30.1 (VDD), LED4.1 (VDD), LED5.1 (VDD), LED6.1 (VDD), LED7.1 (VDD), LED8.1 (VDD), LED9.1 (VDD)
- new net: LED48.2 (DOUT), LED54.3 (DIN)
- new net CURR_LIM: R21.1, U10.5 (ILIM)
- new net LED_Data_5V: LED31.3 (DIN), U9.4
- new net SK6803_EN: R20.1, U10.3 (EN)
- new net SK6803_NFAULT: R19.2, U10.4 (~{FAULT})
Other:
- note added: "NOTE: When USB=500mA, select Rlim = 75k = 74.25k @ 1% = 319mA-401mA range"
- note added: "RGB Current Limiter"
- moved on the sheet: C1, C14, C15, C16, C17, C18, C19, C2, C20, C21, F1, F2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

Commit message: Add files via upload
Parts:
- J2, J6: footprint Connector_USB:USB_C_Receptacle_HRO_TYPE-C-31-M-12 -> PCM_marbastlib-various:USB_C_Receptacle_HRO_TYPE-C-31-M-14
Changed lines of the file:
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@@
       (effects (font (size 1.27 1.27)) (justify right))
     )
-    (property "Footprint" "Connector_USB:USB_C_Receptacle_HRO_TYPE-C-31-M-12" (at 534.035 36.83 0)
+    (property "Footprint" "PCM_marbastlib-various:USB_C_Receptacle_HRO_TYPE-C-31-M-14" (at 534.035 36.83 0)
       (effects (font (size 1.27 1.27)) hide)
     )
@@
       (effects (font (size 1.27 1.27)) (justify right))
     )
-    (property "Footprint" "Connector_USB:USB_C_Receptacle_HRO_TYPE-C-31-M-12" (at -118.745 57.15 0)
-      (effects (font (size 1.27 1.27)) hide)
-    )
+    (property "Footprint" "PCM_marbastlib-various:USB_C_Receptacle_HRO_TYPE-C-31-M-14" (at -118.745 57.15 0)
+      (effects (font (size 1.27 1.27)) hide)
+    )

Commit message: Add files via upload
Parts:
- added C40: 100n, Capacitor_SMD:C_0402_1005Metric, symbol Device:C_Small
- added C41: 100n, Capacitor_SMD:C_0805_2012Metric, symbol Device:C
- added C42, C43, C44, C45, C46, C47, C48: 100u, Capacitor_SMD:C_0402_1005Metric, symbol Device:C_Small
- added R22, R23: 5.1k, Resistor_SMD:R_0805_2012Metric, symbol Device:R
- added R24: 75k, Resistor_SMD:R_0805_2012Metric, symbol Device:R
- added U11: 74AHC1G125, SN74AHC1G125DRLR:DRL5, symbol 74xGxx:74AHC1G125
- added U12: TPS2553DBVR, Package_TO_SOT_SMD:SOT-23-6, symbol Ghoul:TPS2553DBVR
- J1, J7: footprint Connector_JST:JST_SH_SM04B-SRSS-TB_1x04-1MP_P1.00mm_Horizontal -> Connector_JST:JST_SH_BM04B-SRSS-TB_1x04-1MP_P1.00mm_Vertical
Connections:
- net +3V3: now also R3.2; no longer LED1.1 (VDD), LED10.1 (VDD), LED11.1 (VDD), LED12.1 (VDD), LED13.1 (VDD), LED14.1 (VDD), LED15.1 (VDD), LED16.1 (VDD), LED17.1 (VDD), LED18.1 (VDD), LED19.1 (VDD), LED2.1 (VDD), LED20.1 (VDD), LED21.1 (VDD), LED22.1 (VDD), LED23.1 (VDD), LED24.1 (VDD), LED25.1 (VDD), LED26.1 (VDD), LED27.1 (VDD), LED28.1 (VDD), LED29.1 (VDD), LED3.1 (VDD), LED30.1 (VDD), LED4.1 (VDD), LED5.1 (VDD), LED6.1 (VDD), LED7.1 (VDD), LED8.1 (VDD), LED9.1 (VDD)
- net +5V: now also C40.2, C41.1, R22.1, U11.5 (VCC), U12.1 (IN)
- net GND: now also C40.1, C41.2, C42.1, C43.1, C44.1, C45.1, C46.1, C47.1, C48.1, R23.2, R24.2, U11.1, U11.3 (GND), U12.2 (GND)
- net LED_Data_3V3: now also U3.3 (GPIO1); no longer U3.39 (GPIO27_ADC1)
- net LED_Pow_5V: now also C47.2
- net Q_CLK: no longer U7.6 (CLK), U8.52 (QSPI_SCLK)
- net Q_IO0: no longer U7.5 (DI(IO0)), U8.53 (QSPI_SD0)
- net Q_IO1: no longer U7.2 (DO(IO1)), U8.55 (QSPI_SD1)
- net Q_IO2: no longer U7.3 (IO2), U8.54 (QSPI_SD2)
- net Q_IO3: no longer U7.7 (IO3), U8.51 (QSPI_SD3)
- net Q_SEL: no longer R17.1, R18.1, U7.1 (~{CS}), U8.56 (QSPI_SS)
- net R: no longer J3.R, U8.31 (GPIO20)
- net RESET: no longer J8.1 (Pin_1), R16.1, RST2.2, U8.26 (RUN)
- net SWC: no longer J8.4 (Pin_4), U8.24 (SWCLK)
- net SWD: no longer J8.5 (Pin_5), U8.25 (SWD)
- net XIN: no longer C20.2, U8.20 (XIN), Y2.3
- net XOUT: no longer R12.1, U8.21 (XOUT)
- net col 0: no longer SW2.S2, U8.27 (GPIO16)
- net col 1: no longer MX36.1, MX42.1, MX48.1, MX54.1, MX55.1, U8.9 (GPIO7)
- net col 2: no longer MX35.1, MX41.1, MX47.1, MX53.1, MX56.1, U8.11 (GPIO8)
- net col 3: no longer MX33.1, MX40.1, MX46.1, MX52.1, MX59.1, U8.12 (GPIO9)
- net col 4: no longer MX34.1, MX39.1, MX45.1, MX51.1, MX57.1, U8.13 (GPIO10)
- net col 5: no longer MX32.1, MX38.1, MX44.1, MX50.1, MX58.1, U8.14 (GPIO11)
- net col 6: no longer MX31.1, MX42.1, MX43.1, MX49.1, MX60.1, U8.15 (GPIO12)
- net rot A: no longer SW2.A, U8.41 (GPIO29_ADC3)
- net rot B: no longer SW2.B, U8.40 (GPIO28_ADC2)
- net row 0: no longer D32.1 (K), D33.1 (K), D34.1 (K), D35.1 (K), D36.1 (K), D37.1 (K), U8.18 (GPIO15)
- net row 1: no longer D39.1 (K), D40.1 (K), D41.1 (K), D42.1 (K), D43.1 (K), D43.1 (K), U8.36 (GPIO24)
- net row 2: no longer D44.1 (K), D45.1 (K), D46.1 (K), D47.1 (K), D48.1 (K), D49.1 (K), U8.35 (GPIO23)
- net row 3: no longer D50.1 (K), D51.1 (K), D52.1 (K), D53.1 (K), D54.1 (K), D55.1 (K), D62.1 (K), U8.34 (GPIO22)
- net row 4: no longer D56.1 (K), D57.1 (K), D58.1 (K), D59.1 (K), D60.1 (K), D61.1 (K), U8.32 (GPIO21)
- net at LED14.2 (DOUT): now also LED15.3 (DIN); no longer LED13.3 (DIN)
- net at LED14.3 (DIN): now also LED13.2 (DOUT); no longer LED15.2 (DOUT)
- net at LED22.2 (DOUT): now also LED21.3 (DIN); no longer LED23.3 (DIN)
- net at LED22.3 (DIN): now also LED23.2 (DOUT); no longer LED21.2 (DOUT)
- net at LED1.2 (DOUT): now also LED2.3 (DIN)
- net at LED2.2 (DOUT): now also LED3.3 (DIN); no longer LED1.3 (DIN)
- net at LED18.2 (DOUT): now also LED24.3 (DIN); no longer LED17.3 (DIN)
- net at LED18.3 (DIN): now also LED17.2 (DOUT); no longer LED24.2 (DOUT)
- net at LED12.2 (DOUT): now also LED11.3 (DIN); no longer LED6.3 (DIN)
- net at LED12.3 (DIN): now also LED6.2 (DOUT); no longer LED11.2 (DOUT)
- net at LED3.2 (DOUT): now also LED4.3 (DIN); no longer LED2.3 (DIN)
- net at LED4.2 (DOUT): now also LED5.3 (DIN); no longer LED3.3 (DIN)
- net at LED5.2 (DOUT): now also LED6.3 (DIN); no longer LED4.3 (DIN)
- net row 0_L: now reaches U8.2 (GPIO0)
- net row 0_L: now also D32.1 (K), D33.1 (K), D34.1 (K), D35.1 (K), D36.1 (K), D37.1 (K)
- net row 1_L: now reaches U8.29 (GPIO18)
- net row 1_L: now also D39.1 (K), D40.1 (K), D41.1 (K), D42.1 (K), D43.1 (K), D43.1 (K)
- net col 1_L: now reaches U8.3 (GPIO1)
- net col 1_L: now also MX36.1, MX42.1, MX48.1, MX54.1, MX55.1
- net row 2_L: now reaches U8.30 (GPIO19)
- net row 2_L: now also D44.1 (K), D45.1 (K), D46.1 (K), D47.1 (K), D48.1 (K), D49.1 (K)
- net col 2_L: now reaches U8.4 (GPIO2)
- net col 2_L: now also MX35.1, MX41.1, MX47.1, MX53.1, MX56.1
- net col 3_L: now reaches U8.5 (GPIO3)
- net col 3_L: now also MX33.1, MX40.1, MX46.1, MX52.1, MX59.1
- net col 4_L: now reaches U8.6 (GPIO4)
- net col 4_L: now also MX34.1, MX39.1, MX45.1, MX51.1, MX57.1
- net col 5_L: now reaches U8.7 (GPIO5)
- net col 5_L: now also MX32.1, MX38.1, MX44.1, MX50.1, MX58.1
- net at LED8.2 (DOUT): now also LED7.3 (DIN); no longer LED9.3 (DIN)
- net at LED8.3 (DIN): now also LED9.2 (DOUT); no longer LED7.2 (DOUT)
- net at LED20.2 (DOUT): now also LED19.3 (DIN); no longer LED21.3 (DIN)
- net at LED20.3 (DIN): now also LED21.2 (DOUT); no longer LED19.2 (DOUT)
- net at LED28.2 (DOUT): now also LED29.3 (DIN); no longer LED27.3 (DIN)
- net at LED28.3 (DIN): now also LED27.2 (DOUT); no longer LED29.2 (DOUT)
- net at LED10.2 (DOUT): now also LED9.3 (DIN); no longer LED11.3 (DIN)
- net at LED10.3 (DIN): now also LED11.2 (DOUT); no longer LED9.2 (DOUT)
- net at LED30.2 (DOUT): no longer LED29.3 (DIN)
- net at LED25.2 (DOUT): now also LED26.3 (DIN); no longer LED19.3 (DIN)
- net at LED25.3 (DIN): now also LED19.2 (DOUT); no longer LED26.2 (DOUT)
- net at LED16.3 (DIN): now also LED15.2 (DOUT); no longer LED17.2 (DOUT)
- net at LED16.2 (DOUT): now also LED17.3 (DIN); no longer LED15.3 (DIN)
- net LED_Data: no longer names the net of LED30.3 (DIN)
- net LED_Data: now also LED29.2 (DOUT)
- new net: LED23.3 (DIN), LED24.2 (DOUT)
- new net: LED13.3 (DIN), LED7.2 (DOUT)
- new net: LED26.2 (DOUT), LED27.3 (DIN)
- new net CURR_LIM_L: R24.1, U12.5 (ILIM)
- new net LED_Data_3V3_L: U11.2, U8.12 (GPIO9)
- new net LED_Data_5V_L: LED1.3 (DIN), U11.4
- new net LED_Pow_5V_L: C42.2, C43.2, C44.2, C45.2, C46.2, C48.2, LED1.1 (VDD), LED10.1 (VDD), LED11.1 (VDD), LED12.1 (VDD), LED13.1 (VDD), LED14.1 (VDD), LED15.1 (VDD), LED16.1 (VDD), LED17.1 (VDD), LED18.1 (VDD), LED19.1 (VDD), LED2.1 (VDD), LED20.1 (VDD), LED21.1 (VDD), LED22.1 (VDD), LED23.1 (VDD), LED24.1 (VDD), LED25.1 (VDD), LED26.1 (VDD), LED27.1 (VDD), LED28.1 (VDD), LED29.1 (VDD), LED3.1 (VDD), LED30.1 (VDD), LED4.1 (VDD), LED5.1 (VDD), LED6.1 (VDD), LED7.1 (VDD), LED8.1 (VDD), LED9.1 (VDD), U12.6 (OUT)
- new net Q_CLK_L: U7.6 (CLK), U8.52 (QSPI_SCLK)
- new net Q_IO0_L: U7.5 (DI(IO0)), U8.53 (QSPI_SD0)
- new net Q_IO1_L: U7.2 (DO(IO1)), U8.55 (QSPI_SD1)
- new net Q_IO2_L: U7.3 (IO2), U8.54 (QSPI_SD2)
- new net Q_IO3_L: U7.7 (IO3), U8.51 (QSPI_SD3)
- new net Q_SEL_L: R17.1, R18.1, U7.1 (~{CS}), U8.56 (QSPI_SS)
- new net RESET_L: J8.1 (Pin_1), R16.1, RST2.2, U8.26 (RUN)
- new net R_L: J3.R, U8.36 (GPIO24)
- new net SK6803_EN_L: R23.1, U12.3 (EN)
- new net SK6803_NFAULT_L: R22.2, U12.4 (~{FAULT})
- new net SWC_L: J8.4 (Pin_4), U8.24 (SWCLK)
- new net SWD_L: J8.5 (Pin_5), U8.25 (SWD)
- new net XIN_L: C20.2, U8.20 (XIN), Y2.3
- new net XOUT_L: R12.1, U8.21 (XOUT)
- new net col 0_L: SW2.S2, U8.34 (GPIO22)
- new net col 6_L: MX31.1, MX42.1, MX43.1, MX49.1, MX60.1, U8.11 (GPIO8)
- new net rot A_L: SW2.A, U8.41 (GPIO29_ADC3)
- new net rot B_L: SW2.B, U8.40 (GPIO28_ADC2)
- new net row 3_L: D50.1 (K), D51.1 (K), D52.1 (K), D53.1 (K), D54.1 (K), D55.1 (K), D62.1 (K), U8.31 (GPIO20)
- new net row 4_L: D56.1 (K), D57.1 (K), D58.1 (K), D59.1 (K), D60.1 (K), D61.1 (K), U8.32 (GPIO21)
Other:
- moved on the sheet: BOOT1, BOOT2, C1, C10, C11, C12, C13, C14, C15, C16, C17, C18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
