File: Chastity/chastity.kicad_sch (KiCad schematic)
At the start: 284 parts, among them J10 USB_C_Receptacle_USB2.0, J2 USB_C_Receptacle_USB2.0, J4 Conn_01x05, J6 USB_C_Receptacle_USB2.0, J8 Conn_01x05, J9 USB_C_Receptacle_USB2.0_L, SW2 RotaryEncoder_Switch, U1 XC6206PxxxMR, U10 TPS2553DBVR, U11 74AHC1G125, U12 TPS2553DBVR, U2 SRV05-4, U3 RP2040, U4 W25Q128JVS, U5 XC6206PxxxMR, U6 SRV05-4, U7 W25Q128JVS, U8 RP2040, U9 74AHC1G125, Y1 Crystal_GND24, Y2 Crystal_GND24

Commit message: Add files via upload
Parts:
- removed J10: USB_C_Receptacle_USB2.0, PCM_marbastlib-various:USB_C_Receptacle_HRO_TYPE-C-31-M-14, symbol Connector:USB_C_Receptacle_USB2.0
- removed J9: USB_C_Receptacle_USB2.0_L, PCM_marbastlib-various:USB_C_Receptacle_HRO_TYPE-C-31-M-14, symbol Connector:USB_C_Receptacle_USB2.0
- added R25, R26, R27, R28: 5K1, Resistor_SMD:R_0402_1005Metric, symbol Device:R_Small
- added SPLIT1 (x2): USB-C-2.0, Connector_USB:USB_C_Receptacle_HRO_TYPE-C-31-M-12, symbol Connector:USB_C_Receptacle_USB2.0
- J4, J8: footprint Connector_PinSocket_2.54mm:PinSocket_1x05_P2.54mm_Vertical -> Connector_PinSocket_2.54mm:PinSocket_1x05_P2.54mm_Horizontal
Connections:
- net GND: now also R25.2, R26.2, R27.2, R28.2, SPLIT1.A1 (GND), SPLIT1.A1 (GND), SPLIT1.A12 (GND), SPLIT1.A12 (GND), SPLIT1.B1 (GND), SPLIT1.B1 (GND), SPLIT1.B12 (GND), SPLIT1.B12 (GND), SPLIT1.S1 (SHIELD), SPLIT1.S1 (SHIELD)
- net VBUS: now also SPLIT1.A4 (VBUS), SPLIT1.A4 (VBUS), SPLIT1.A9 (VBUS), SPLIT1.A9 (VBUS), SPLIT1.B4 (VBUS), SPLIT1.B4 (VBUS), SPLIT1.B9 (VBUS), SPLIT1.B9 (VBUS)
- net D_Split_L-: now reaches U8.16 (GPIO13)
- net D_Split_L-: now also SPLIT1.A7 (D-), SPLIT1.B7 (D-)
- net D_Split_L+: now reaches U8.17 (GPIO14)
- net D_Split_L+: now also SPLIT1.A6 (D+), SPLIT1.B6 (D+)
- net D_Split_R-: now reaches U3.5 (GPIO3)
- net D_Split_R-: now also SPLIT1.A7 (D-), SPLIT1.B7 (D-)
- net D_Split_R+: now reaches U3.6 (GPIO4)
- net D_Split_R+: now also SPLIT1.A6 (D+), SPLIT1.B6 (D+)
- new net: R25.1, SPLIT1.A5 (CC1)
- new net: R26.1, SPLIT1.B5 (CC2)
- new net: R28.1, SPLIT1.B5 (CC2)
- new net: R27.1, SPLIT1.A5 (CC1)
- no-connect marks 8 -> 12

Commit message: Add files via upload
Other:
- moved on the sheet: BOOT1, BOOT2, C1, C10, C11, C12, C13, C14, C15, C16, C17, C18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
