File: V2.5/chastity.kicad_sch (KiCad schematic)
At the start: 290 parts, among them J1 Conn_01x08_Pin, J2 USB_C_Receptacle_USB2.0, J3 Conn_01x08_Pin, J4 Conn_01x05, J6 USB_C_Receptacle_USB2.0, J8 Conn_01x05, SW2 RotaryEncoder_Switch, U1 XC6206PxxxMR, U10 TPS2553DBVR, U11 74AHC1G125, U12 TPS2553DBVR, U2 SRV05-4, U3 RP2040, U4 W25Q128JVS, U5 XC6206PxxxMR, U6 SRV05-4, U7 W25Q128JVS, U8 RP2040, U9 74AHC1G125, Y1 Crystal_GND24, Y2 Crystal_GND24

Commit message: Add files via upload
Parts:
- J2, J6: footprint PCM_marbastlib-various:USB_C_Receptacle_HRO_TYPE-C-31-M-12 -> PCM_marbastlib-various:USB_C_Receptacle_HRO_TYPE-C-31-M-14
- SPLIT1: footprint Connector_USB:USB_C_Receptacle_HRO_TYPE-C-31-M-12 -> Connector_USB:USB_C_Receptacle_HRO_TYPE-C-31-M-14
Changed lines of the file:
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@@
       (effects (font (size 1.27 1.27)) (justify right))
     )
-    (property "Footprint" "PCM_marbastlib-various:USB_C_Receptacle_HRO_TYPE-C-31-M-12" (at 46.355 61.595 0)
+    (property "Footprint" "PCM_marbastlib-various:USB_C_Receptacle_HRO_TYPE-C-31-M-14" (at 46.355 61.595 0)
       (effects (font (size 1.27 1.27)) hide)
     )
@@
       (effects (font (size 1.27 1.27)) (justify right))
     )
-    (property "Footprint" "PCM_marbastlib-various:USB_C_Receptacle_HRO_TYPE-C-31-M-12" (at 47.625 223.52 0)
+    (property "Footprint" "PCM_marbastlib-various:USB_C_Receptacle_HRO_TYPE-C-31-M-14" (at 47.625 223.52 0)
       (effects (font (size 1.27 1.27)) hide)
     )
@@
       (effects (font (size 1.27 1.27)))
     )
-    (property "Footprint" "Connector_USB:USB_C_Receptacle_HRO_TYPE-C-31-M-12" (at 528.32 51.435 0)
+    (property "Footprint" "Connector_USB:USB_C_Receptacle_HRO_TYPE-C-31-M-14" (at 528.32 51.435 0)
       (effects (font (size 1.27 1.27)) hide)
     )
@@
       (effects (font (size 1.27 1.27)))
     )
-    (property "Footprint" "Connector_USB:USB_C_Receptacle_HRO_TYPE-C-31-M-12" (at 528.955 179.07 0)
+    (property "Footprint" "Connector_USB:USB_C_Receptacle_HRO_TYPE-C-31-M-14" (at 528.955 179.07 0)
       (effects (font (size 1.27 1.27)) hide)
     )

Commit message: Add files via upload
Parts:
- removed C34, C35, C36, C37, C38, C42, C43, C44, C45, C47, C48: 100u, Capacitor_SMD:C_0402_1005Metric, symbol Device:C_Small
- added C101, C102, C103, C104, C105, C106, C107, C108, C109, C110, C111, C112, C113, C114, C115, C116, C117, C118, C119, C120, C121, C122, C123, C124, C125, C127, C128, C129, C130, C131, C132, C133, C134, C135, C136, C137, C138, C139, C140, C141, C142, C143, C144, C145, C146, C147, C148, C149, C150, C151, C152, C153, C154, C155, C156, C157, C158, C159, C160: 100n, Capacitor_SMD:C_0402_1005Metric, symbol Device:C_Small
- added TFT101, TFT102: ~, 505110-1292:TFT 1.47 waveshare, symbol PCM_marbastlib-promicroish:TFT_1.47
- C126: renamed from C46; value 100u -> 100n
- C39, C41: footprint Capacitor_SMD:C_0805_2012Metric -> Capacitor_SMD:C_0402_1005Metric
- R19, R20, R22, R23: value 5.1k -> 5k1; footprint Resistor_SMD:R_0805_2012Metric -> Resistor_SMD:R_0402_1005Metric
- R21, R24: footprint Resistor_SMD:R_0805_2012Metric -> Resistor_SMD:R_0402_1005Metric
- SPLIT1: value USB-C-2.0 -> USB_C_Receptacle_USB2.0; footprint Connector_USB:USB_C_Receptacle_HRO_TYPE-C-31-M-14 -> PCM_marbastlib-various:USB_C_Receptacle_HRO_TYPE-C-31-M-14
Connections:
- net D+: no longer J2.A6 (D+), J2.B6 (D+), R13.2, U6.1 (IO1)
- net D-: no longer J2.A7 (D-), J2.B7 (D-), R14.2, U6.6 (IO4)
- net GND: now also C101.1, C102.1, C103.1, C104.1, C105.1, C106.1, C107.1, C108.1, C109.1, C110.1, C111.1, C112.1, C113.1, C114.1, C115.1, C116.1, C117.1, C118.1, C119.1, C120.1, C121.1, C122.1, C123.1, C124.1, C125.1, C127.1, C128.1, C129.1, C130.1, C131.1, C132.1, C133.1, C134.1, C135.1, C136.1, C137.1, C138.1, C139.1, C140.1, C141.1, C142.1, C143.1, C144.1, C145.1, C146.1, C147.1, C148.1, C149.1, C150.1, C151.1, C152.1, C153.1, C154.1, C155.1, C156.1, C157.1, C158.1, C159.1, C160.1
- net LED_Pow_5V: now also C131.2, C132.2, C133.2, C134.2, C135.2, C136.2, C137.2, C138.2, C139.2, C140.2, C141.2, C142.2, C143.2, C144.2, C145.2, C146.2, C147.2, C148.2, C149.2, C150.2, C151.2, C152.2, C153.2, C154.2, C155.2, C156.2, C157.2, C158.2, C159.2, C160.2
- net LED_Pow_5V_L: now also C101.2, C102.2, C103.2, C104.2, C105.2, C106.2, C107.2, C108.2, C109.2, C110.2, C111.2, C112.2, C113.2, C114.2, C115.2, C116.2, C117.2, C118.2, C119.2, C120.2, C121.2, C122.2, C123.2, C124.2, C125.2, C127.2, C128.2, C129.2, C130.2
- new net DL+: J2.A6 (D+), J2.B6 (D+), R13.2, U6.1 (IO1)
- new net DL-: J2.A7 (D-), J2.B7 (D-), R14.2, U6.6 (IO4)
Other:
- note added: "TFT & Connector"
- note removed: "TFT connector"
- moved on the sheet: C126, J1, J3
